Commit message: 修改：仿真模型
1. 移动机器人放置在铁塔下方
2. 激光雷达高度调高

File: urdf/livox_avia.xacro (robot description, xacro)
@@ -11,5 +11,5 @@
   <xacro:macro name="null_inertial">
     <inertial>
-      <mass value="0.1"/>
+      <mass value="0.0"/>
     <inertia ixx="0.01" ixy="0" ixz="0"
           iyy="0.01" iyz="0"
@@ -64,5 +64,4 @@
       <xacro:null_inertial/>
       <visual>
-      <!-- 位置和姿态 -->
         <origin xyz="0.00 0 0.00" rpy="0 0 0"/>
         <geometry>

File: urdf/standardrobots_oasis300.xacro (robot description, xacro)
@@ -51,5 +51,5 @@
 		<parent link="${world_link}"/>
 		<child link="${base_link}"/>
-		<origin xyz="0.0 0 0.05" rpy="0 0 ${M_PI/2}" />
+		<origin xyz="0.0 -17 0" rpy="0 0 0" />
 	</joint>
 	<joint name="livox_base_joint" type="fixed">
@@ -57,5 +57,5 @@
         <child link="livox_base"/>
         <origin rpy="0 0 1.5707"
-                xyz="0.0 0.4 0.3057"/>
+                xyz="0.0 0.4 20"/>
     </joint>
     </xacro:macro>
